Commit message: Pinch where the thumb meets the index finger, not at the power-grasp frame
The grasp was planned for {side}_hand_grasp_frame, a power-grasp estimate; from the hand's own
finger kinematics the thumb and index tips meet 4.7/4.5/2.9 cm from it, so the pinch closed
beside the panel.

- g1_description: {side}_hand_pinch_frame at that meeting point.
- Pick/Place plan published grasps for the pinch frame.
- SRDF pinch_open: thumb across, thumb and fingers 40 % closed (straight fingers reached 6.5 cm
  past the point into the panel's inside).
- Panel grasp point moved into the edge's lip (z +35 mm, measured on the STL); the RViz hand
  is drawn in the pinch_open shape around the point.

Co-Authored-By: Claude Opus 5.5 <noreply@anthropic.com>
Claude-Session: https://claude.ai/code/session_01JXseFTqZS9kKoE3DMXGb5q

File: workspace/src/g1_description/urdf/g1_arm_sdk.urdf.xacro (robot description, xacro)
@@ -198,3 +198,14 @@
   <xacro:g1_grasp_frame side="left"/>
   <xacro:g1_grasp_frame side="right"/>
+  <!-- Where a thumb-to-index pinch closes. See pinch_frame in config/rh56e2_params.yaml. -->
+  <xacro:macro name="g1_pinch_frame" params="side">
+    <link name="${side}_hand_pinch_frame"/>
+    <joint name="${side}_hand_pinch_frame_joint" type="fixed">
+      <parent link="${side}_hand_palm_link"/>
+      <child link="${side}_hand_pinch_frame"/>
+      <origin xyz="${rh56e2_params.pinch_frame[side].xyz}" rpy="0 0 0"/>
+    </joint>
+  </xacro:macro>
+  <xacro:g1_pinch_frame side="left"/>
+  <xacro:g1_pinch_frame side="right"/>
 </robot>
